File: Schematics/sensor/Caleb_version/PCB_Sensor.brd (EAGLE design)
At the start: 29.6 x 28.2 mm, 21 parts, among them U1 ATMEGA328P

Commit message: Revision by Caleb
Changed programming connectors to be on the surface as pads only for
programming with another board.
Rearranged the board to minimize the size as much as possible.
Dimensions are .95 x .65
Parts:
- removed D11, D12, D13, GND, RST, VCC: M01SMD, SparkFun-Connectors:LUXEON-PAD
- added JP1, JP2: M01POGOPIN_HOLE_0.58, SparkFun-Connectors:1X01_POGOPIN_HOLE_0.58
- added U$1: POGOPIN-BACKBOARD, Protofusion:POGOPROG-BACKMOUNT
- added U$2: POGOPIN-CONNSTANDARD, Protofusion:POGOPROG-CONN
Connections:
- net D11: now also U$2.2; no longer D11.P$1
- net D12: now also U$2.3; no longer D12.P$1
- net D13: now also U$2.4; no longer D13.P$1
- net GND: now also U$2.5; no longer GND.P$1
- net RST: now also U$2.1; no longer RST.P$1
- net VCC: now also U$2.6; no longer VCC.P$1
