File: Schematics/sensor/Caleb_version/PCB_Sensor.sch (EAGLE design)
At the start: 21 parts, among them U1 ATMEGA328P

Commit message: Revision by Caleb
Changed programming connectors to be on the surface as pads only for
programming with another board.
Rearranged the board to minimize the size as much as possible.
Dimensions are .95 x .65
Parts:
- removed D11, D12, D13, GND, RST, VCC: M01SMD, SparkFun-Connectors:M01SMD
- added JP1, JP2: M01POGOPIN_HOLE_0.58, SparkFun-Connectors:M01POGOPIN_HOLE_0.58
- added U$1: POGOPIN-BACKBOARD, Protofusion:POGOPIN-BACKBOARD
- added U$2: POGOPIN-CONNSTANDARD, Protofusion:POGOPIN-CONNSTANDARD
Connections:
- net D11: now also U$2.MOSI; no longer D11.1
- net D12: now also U$2.MISO; no longer D12.1
- net D13: now also U$2.SCK; no longer D13.1
- net GND: now also U$2.GND; no longer GND.1
- net RST: now also U$2.\RST; no longer RST.1
- net VCC: now also U$2.VCC; no longer VCC.1
Changed lines of the file:
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@@
 <layer number="108" name="tplace-old" color="10" fill="1" visible="yes" active="yes"/>
 <layer number="109" name="ref-old" color="11" fill="1" visible="yes" active="yes"/>
+<layer number="111" name="tGTest" color="7" fill="1" visible="yes" active="yes"/>
+<layer number="112" name="bGTest" color="7" fill="1" visible="yes" active="yes"/>
 <layer number="116" name="Patch_BOT" color="9" fill="4" visible="yes" active="yes"/>
+<layer number="117" name="mPads" color="7" fill="1" visible="yes" active="yes"/>
+<layer number="118" name="mVias" color="7" fill="1" visible="yes" active="yes"/>
+<layer number="119" name="mUnrouted" color="7" fill="1" visible="yes" active="yes"/>
+<layer number="120" name="mDimension" color="7" fill="1" visible="yes" active="yes"/>
 <layer number="121" name="_tsilk" color="7" fill="1" visible="yes" active="yes"/>
 <layer number="122" name="_bsilk" color="7" fill="1" visible="yes" active="yes"/>
+<layer number="123" name="mtOrigins" color="7" fill="1" visible="yes" active="yes"/>
+<layer number="124" name="mbOrigins" color="7" fill="1" visible="yes" active="yes"/>
 <layer number="125" name="_tNames" color="7" fill="1" visible="yes" active="yes"/>
+<layer number="126" name="_bNames" color="7" fill="1" visible="yes" active="yes"/>
+<layer number="127" name="mtValues" color="7" fill="1" visible="yes" active="yes"/>
+<layer number="128" name="mbValues" color="7" fill="1" visible="yes" active="yes"/>
+<layer number="129" name="mtStop" color="7" fill="1" visible="yes" active="yes"/>
+<layer number="130" name="mbStop" color="7" fill="1" visible="yes" active="yes"/>
+<layer number="131" name="prix" color="7" fill="1" visible="yes" active="yes"/>
+<layer number="132" name="test" color="7" fill="1" visible="yes" active="yes"/>
+<layer number="133" name="mtFinish" color="7" fill="1" visible="yes" active="yes"/>
+<layer number="134" name="mbFinish" color="7" fill="1" visible="yes" active="yes"/>
+<layer number="135" name="mtGlue" color="7" fill="1" visible="yes" active="yes"/>
+<layer number="136" name="mbGlue" color="7" fill="1" visible="yes" active="yes"/>
+<layer number="137" name="mtTest" color="7" fill="1" visible="yes" active="yes"/>
+<layer number="138" name="mbTest" color="7" fill="1" visible="yes" active="yes"/>
+<layer number="139" name="mtKeepout" color="7" fill="1" visible="yes" active="yes"/>
+<layer number="140" name="mbKeepout" color="7" fill="1" visible="yes" active="yes"/>
+<layer number="141" name="mtRestrict" color="7" fill="1" visible="yes" active="yes"/>
+<layer number="142" name="mbRestrict" color="7" fill="1" visible="yes" active="yes"/>
+<layer number="143" name="mvRestrict" color="7" fill="1" visible="yes" active="yes"/>
 <layer number="144" name="Drill_legend" color="7" fill="1" visible="yes" active="yes"/>
+<layer number="145" name="mHoles" color="7" fill="1" visible="yes" active="yes"/>
+<layer number="146" name="mMilling" color="7" fill="1" visible="yes" active="yes"/>
+<layer number="147" name="mMeasures" color="7" fill="1" visible="yes" active="yes"/>
+<layer number="148" name="mDocument" color="7" fill="1" visible="yes" active="yes"/>
+<layer number="149" name="mReference" color="7" fill="1" visible="yes" active="yes"/>
+<layer number="150" name="Notes" color="7" fill="1" visible="yes" active="yes"/>
 <layer number="151" name="HeatSink" color="7" fill="1" visible="yes" active="yes"/>
+<layer number="152" name="mbDocu" color="7" fill="1" visible="yes" active="yes"/>
+<layer number="191" name="mNets" color="7" fill="1" visible="yes" active="yes"/>
+<layer number="192" name="mBusses" color="7" fill="1" visible="yes" active="yes"/>
+<layer number="193" name="mPins" color="7" fill="1" visible="yes" active="yes"/>
+<layer number="194" name="mSymbols" color="7" fill="1" visible="yes" active="yes"/>
+<layer number="195" name="mNames" color="7" fill="1" visible="yes" active="yes"/>
+<layer number="196" name="mValues" color="7" fill="1" visible="yes" active="yes"/>
 <layer number="199" name="Contour" color="7" fill="1" visible="yes" active="yes"/>
 <layer number="200" name="200bmp" color="1" fill="10" visible="yes" active="yes"/>
@@
 <layer number="251" name="SMDround" color="12" fill="11" visible="no" active="no"/>
 <layer number="254" name="cooling" color="7" fill="1" visible="yes" active="yes"/>
+<layer number="255" name="PART_" color="7" fill="1" visible="yes" active="yes"/>
 </layers>
 <schematic xreflabel="%F%N/%S.%C%R" xrefpart="/%S.%C%R">
@@
 <part name="RX" library="SparkFun-Connectors" deviceset="M01" device="SMD"/>
 <part name="TX" library="SparkFun-Connectors" deviceset="M01" device="SMD"/>
-<part name="D13" library="SparkFun-Connectors" deviceset="M01" device="SMD"/>
-<part name="D12" library="SparkFun-Connectors" deviceset="M01" device="SMD"/>
-<part name="RST" library="SparkFun-Connectors" deviceset="M01" device="SMD"/>
-<part name="D11" library="SparkFun-Connectors" deviceset="M01" device="SMD"/>
-<part name="VCC" library="SparkFun-Connectors" deviceset="M01" device="SMD"/>
-<part name="GND" library="SparkFun-Connectors" deviceset="M01" device="SMD"/>
 <part name="GND2" library="SparkFun-Aesthetics" deviceset="GND" device=""/>
 <part name="GND3" library="SparkFun-Aesthetics" deviceset="GND" device=""/>
 <part name="GND4" library="SparkFun-Aesthetics" deviceset="GND" device=""/>
 <part name="GND5" library="SparkFun-Aesthetics" deviceset="GND" device=""/>
+<part name="U$1" library="Protofusion" deviceset="POGOPIN-BACKBOARD" device=""/>
+<part name="U$2" library="Protofusion" deviceset="POGOPIN-CONN" device="STANDARD"/>
+<part name="JP1" library="SparkFun-Connectors" deviceset="M01" device="POGOPIN_HOLE_0.58"/>
+<part name="JP2" library="SparkFun-Connectors" deviceset="M01" device="POGOPIN_HOLE_0.58"/>
 </parts>
 <sheets>
@@
 <instance part="RX" gate="G$1" x="-2.54" y="119.38"/>
 <instance part="TX" gate="G$1" x="-2.54" y="109.22"/>
-<instance part="D13" gate="G$1" x="78.74" y="96.52" rot="R180"/>
-<instance part="D12" gate="G$1" x="78.74" y="106.68" rot="R180"/>
-<instance part="RST" gate="G$1" x="78.74" y="86.36" rot="R180"/>
-<instance part="D11" gate="G$1" x="86.36" y="96.52"/>
-<instance part="VCC" gate="G$1" x="86.36" y="106.68"/>
-<instance part="GND" gate="G$1" x="86.36" y="86.36"/>
 <instance part="GND2" gate="1" x="152.4" y="111.76"/>
 <instance part="GND3" gate="1" x="27.94" y="132.08"/>
 <instance part="GND4" gate="1" x="10.16" y="132.08"/>
 <instance part="GND5" gate="1" x="43.18" y="96.52"/>
+<instance part="U$1" gate="G$1" x="20.32" y="71.12"/>
+<instance part="U$2" gate="J" x="73.66" y="101.6"/>
+<instance part="JP1" gate="G$1" x="114.3" y="99.06"/>
+<instance part="JP2" gate="G$1" x="114.3" y="88.9"/>
 </instances>
 <busses>
@@
 </segment>
 <segment>
-<wire x1="93.98" y1="86.36" x2="101.6" y2="86.36" width="0.1524" layer="91"/>
-<label x="96.52" y="86.36" size="1.778" layer="95"/>
-<pinref part="GND" gate="G$1" pin="1"/>
+<wire x1="63.5" y1="104.14" x2="71.12" y2="104.14" width="0.1524" layer="91"/>
+<label x="63.5" y="104.14" size="1.778" layer="95"/>
+<pinref part="U$2" gate="J" pin="GND"/>
 </segment>
 <segment>
@@
 </segment>
 <segment>
-<wire x1="93.98" y1="106.68" x2="101.6" y2="106.68" width="0.1524" layer="91"/>
-<label x="96.52" y="106.68" size="1.778" layer="95"/>
-<pinref part="VCC" gate="G$1" pin="1"/>
+<wire x1="63.5" y1="106.68" x2="71.12" y2="106.68" width="0.1524" layer="91"/>
+<label x="63.5" y="106.68" size="1.778" layer="95"/>
+<pinref part="U$2" gate="J" pin="VCC"/>
 </segment>
 <segment>
@@
 </segment>
 <segment>
-<wire x1="71.12" y1="86.36" x2="63.5" y2="86.36" width="0.1524" layer="91"/>
-<label x="63.5" y="86.36" size="1.778" layer="95"/>
-<pinref part="RST" gate="G$1" pin="1"/>
+<wire x1="71.12" y1="93.98" x2="63.5" y2="93.98" width="0.1524" layer="91"/>
+<label x="63.5" y="93.98" size="1.778" layer="95"/>
+<pinref part="U$2" gate="J" pin="\RST"/>
 </segment>
 </net>
@@
 </segment>
 <segment>
-<wire x1="71.12" y1="96.52" x2="63.5" y2="96.52" width="0.1524" layer="91"/>
-<label x="63.5" y="96.52" size="1.778" layer="95"/>
-<pinref part="D13" gate="G$1" pin="1"/>
+<wire x1="71.12" y1="101.6" x2="63.5" y2="101.6" width="0.1524" layer="91"/>
+<label x="63.5" y="101.6" size="1.778" layer="95"/>
+<pinref part="U$2" gate="J" pin="SCK"/>
 </segment>
 </net>
@@
 </segment>
 <segment>
-<wire x1="71.12" y1="106.68" x2="63.5" y2="106.68" width="0.1524" layer="91"/>
-<label x="63.5" y="106.68" size="1.778" layer="95"/>
-<pinref part="D12" gate="G$1" pin="1"/>
+<wire x1="71.12" y1="99.06" x2="63.5" y2="99.06" width="0.1524" layer="91"/>
+<label x="63.5" y="99.06" size="1.778" layer="95"/>
+<pinref part="U$2" gate="J" pin="MISO"/>
 </segment>
 </net>
@@
 </segment>
 <segment>
-<wire x1="93.98" y1="96.52" x2="101.6" y2="96.52" width="0.1524" layer="91"/>
-<label x="96.52" y="96.52" size="1.778" layer="95"/>
-<pinref part="D11" gate="G$1" pin="1"/>
-</segment>
-</net>
+<wire x1="63.5" y1="96.52" x2="71.12" y2="96.52" width="0.1524" layer="91"/>
+<label x="63.5" y="96.52" size="1.778" layer="95"/>
+<pinref part="U$2" gate="J" pin="MOSI"/>
+</segment>
+</net>
