File: Schematics/sensor/sensor.sch (EAGLE design)
At the start: 16 parts, among them Y1 16MHz

Commit message: PCB improvements
Node_SP 2.0: moved some text to the back layer

Sen_SP 4.0: improved the board for programming and changed the
resonator from through hole to surface mount - then rearranged the
items on the board to make it smaller
Parts:
- removed 15P, 16P, 17P, 5VP, GP, RST, RX, TX: PTR1TP12R, testpad:PTR1TP12R
- removed Y1: 16MHz, SparkFun-FreqCtrl:RESONATORPTH
- added PAD3, PAD4, PAD5, PAD6, PAD7, PAD8: (no value), wirepad:1,6/0,9
- added Y2: 16MHz, SparkFun-FreqCtrl:RESONATOR16MHZ
Connections:
- removed net N$3: 17P.TP, ATMEGA328P.PB5(SCK)
- removed net N$4: 16P.TP, ATMEGA328P.PB4(MISO)
- removed net N$5: 15P.TP, ATMEGA328P.PB3(MOSI/OC2)
- new net 1: ATMEGA328P.PB4(MISO), PAD5.P
- new net 3: ATMEGA328P.PB5(SCK), PAD4.P
- new net 4: ATMEGA328P.PB3(MOSI/OC2), PAD6.P
- net 5V: now also PAD7.P; no longer 5VP.TP
- net GND: now also PAD1.P, Y2.2; no longer GP.TP, Y1.2
- net N$1: now also Y2.1; no longer Y1.1
- net N$2: now also Y2.3; no longer Y1.3
- net N$6: now also PAD3.P; no longer RX.TP
- net N$9: now also PAD2.P; no longer TX.TP
- net RESET: now also PAD8.P; no longer RST.TP
Other:
- moved on the sheet: PAD1, PAD2
Changed lines of the file:
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@@
 <part name="ATMEGA328P" library="SparkFun-DigitalIC" deviceset="ATMEGA328_SMT" device="" value="ATMEGA328P"/>
 <part name="MAX485" library="Maxim_By_element14_Batch_1" deviceset="MAX485CSA+" device=""/>
-<part name="Y1" library="SparkFun-FreqCtrl" deviceset="RESONATOR" device="PTH" value="16MHz"/>
 <part name="GND1" library="SparkFun-Aesthetics" deviceset="GND" device=""/>
 <part name="GND2" library="SparkFun-Aesthetics" deviceset="GND" device=""/>
@@
 <part name="GND6" library="SparkFun-Aesthetics" deviceset="GND" device=""/>
 <part name="SUPPLY6" library="SparkFun-Aesthetics" deviceset="5V" device=""/>
-<part name="15P" library="testpad" deviceset="PTR1" device="TP12R"/>
-<part name="17P" library="testpad" deviceset="PTR1" device="TP12R"/>
-<part name="RST" library="testpad" deviceset="PTR1" device="TP12R"/>
-<part name="16P" library="testpad" deviceset="PTR1" device="TP12R"/>
-<part name="5VP" library="testpad" deviceset="PTR1" device="TP12R"/>
-<part name="GP" library="testpad" deviceset="PTR1" device="TP12R"/>
-<part name="TX" library="testpad" deviceset="PTR1" device="TP12R"/>
-<part name="RX" library="testpad" deviceset="PTR1" device="TP12R"/>
 <part name="JP1" library="SparkFun-Connectors" deviceset="M04" device="PTH"/>
 <part name="JP2" library="SparkFun-Connectors" deviceset="M04" device="PTH"/>
@@
 <part name="PAD1" library="wirepad" deviceset="1,6/0,9" device=""/>
 <part name="PAD2" library="wirepad" deviceset="1,6/0,9" device=""/>
+<part name="PAD3" library="wirepad" deviceset="1,6/0,9" device=""/>
+<part name="PAD4" library="wirepad" deviceset="1,6/0,9" device=""/>
+<part name="PAD5" library="wirepad" deviceset="1,6/0,9" device=""/>
+<part name="PAD6" library="wirepad" deviceset="1,6/0,9" device=""/>
+<part name="PAD7" library="wirepad" deviceset="1,6/0,9" device=""/>
+<part name="PAD8" library="wirepad" deviceset="1,6/0,9" device=""/>
+<part name="Y2" library="SparkFun-FreqCtrl" deviceset="RESONATOR" device="16MHZ" value="16MHz"/>
 </parts>
 <sheets>
@@
 <instance part="ATMEGA328P" gate="G$1" x="48.26" y="93.98"/>
 <instance part="MAX485" gate="A" x="165.1" y="111.76"/>
-<instance part="Y1" gate="G$1" x="22.86" y="91.44" rot="R270"/>
 <instance part="GND1" gate="1" x="10.16" y="88.9"/>
 <instance part="GND2" gate="1" x="147.32" y="96.52"/>
@@
 <instance part="GND6" gate="1" x="200.66" y="101.6"/>
 <instance part="SUPPLY6" gate="G$1" x="22.86" y="132.08"/>
-<instance part="15P" gate="G$1" x="144.78" y="63.5"/>
-<instance part="17P" gate="G$1" x="134.62" y="58.42"/>
-<instance part="RST" gate="G$1" x="129.54" y="55.88"/>
-<instance part="16P" gate="G$1" x="139.7" y="60.96"/>
-<instance part="5VP" gate="G$1" x="86.36" y="43.18"/>
-<instance part="GP" gate="G$1" x="104.14" y="50.8"/>
-<instance part="TX" gate="G$1" x="91.44" y="91.44"/>
-<instance part="RX" gate="G$1" x="96.52" y="93.98"/>
 <instance part="JP1" gate="G$1" x="215.9" y="111.76" rot="R180"/>
 <instance part="JP2" gate="G$1" x="165.1" y="154.94" rot="R180"/>
 <instance part="R2" gate="G$1" x="22.86" y="127" rot="R90"/>
-<instance part="PAD1" gate="1" x="99.06" y="119.38"/>
-<instance part="PAD2" gate="1" x="88.9" y="127"/>
+<instance part="PAD1" gate="1" x="104.14" y="43.18" rot="R90"/>
+<instance part="PAD2" gate="1" x="91.44" y="83.82" rot="R90"/>
+<instance part="PAD3" gate="1" x="96.52" y="83.82" rot="R90"/>
+<instance part="PAD4" gate="1" x="134.62" y="50.8" rot="R90"/>
+<instance part="PAD5" gate="1" x="139.7" y="50.8" rot="R90"/>
+<instance part="PAD6" gate="1" x="144.78" y="50.8" rot="R90"/>
+<instance part="PAD7" gate="1" x="86.36" y="43.18" rot="R90"/>
+<instance part="PAD8" gate="1" x="129.54" y="50.8" rot="R90"/>
+<instance part="Y2" gate="G$1" x="22.86" y="91.44" rot="R270"/>
 </instances>
 <busses>
@@
 <net name="GND" class="0">
 <segment>
-<pinref part="Y1" gate="G$1" pin="2"/>
 <pinref part="GND1" gate="1" pin="GND"/>
 <wire x1="15.24" y1="91.44" x2="10.16" y2="91.44" width="0.1524" layer="91"/>
+<pinref part="Y2" gate="G$1" pin="2"/>
 </segment>
 <segment>
@@
 <segment>
 <pinref part="GND3" gate="1" pin="GND"/>
-<pinref part="GP" gate="G$1" pin="TP"/>
 <wire x1="96.52" y1="53.34" x2="104.14" y2="53.34" width="0.1524" layer="91"/>
+<pinref part="PAD1" gate="1" pin="P"/>
+<wire x1="104.14" y1="45.72" x2="104.14" y2="53.34" width="0.1524" layer="91"/>
 </segment>
 <segment>
@@
 <pinref part="SUPPLY2" gate="G$1" pin="5V"/>
 <wire x1="86.36" y1="45.72" x2="86.36" y2="50.8" width="0.1524" layer="91"/>
-<pinref part="5VP" gate="G$1" pin="TP"/>
+<pinref part="PAD7" gate="1" pin="P"/>
 </segment>
 <segment>
@@
 <net name="N$1" class="0">
 <segment>
-<pinref part="Y1" gate="G$1" pin="1"/>
 <pinref part="ATMEGA328P" gate="G$1" pin="PB6(XTAL1/TOSC1)"/>
 <wire x1="22.86" y1="93.98" x2="25.4" y2="93.98" width="0.1524" layer="91"/>
+<pinref part="Y2" gate="G$1" pin="1"/>
 </segment>
 </net>
 <net name="N$2" class="0">
 <segment>
-<pinref part="Y1" gate="G$1" pin="3"/>
 <pinref part="ATMEGA328P" gate="G$1" pin="PB7(XTAL2/TOSC2)"/>
 <wire x1="22.86" y1="88.9" x2="25.4" y2="88.9" width="0.1524" layer="91"/>
-</segment>
-</net>
-<net name="N$3" class="0">
+<pinref part="Y2" gate="G$1" pin="3"/>
+</segment>
+</net>
+<net name="3" class="0">
 <segment>
 <pinref part="ATMEGA328P" gate="G$1" pin="PB5(SCK)"/>
 <wire x1="73.66" y1="60.96" x2="134.62" y2="60.96" width="0.1524" layer="91"/>
-<pinref part="17P" gate="G$1" pin="TP"/>
-</segment>
-</net>
-<net name="N$4" class="0">
+<pinref part="PAD4" gate="1" pin="P"/>
+<wire x1="134.62" y1="53.34" x2="134.62" y2="60.96" width="0.1524" layer="91"/>
+<label x="114.3" y="60.96" size="1.778" layer="95"/>
+</segment>
+</net>
+<net name="1" class="0">
 <segment>
 <pinref part="ATMEGA328P" gate="G$1" pin="PB4(MISO)"/>
 <wire x1="73.66" y1="63.5" x2="139.7" y2="63.5" width="0.1524" layer="91"/>
-<pinref part="16P" gate="G$1" pin="TP"/>
-</segment>
-</net>
-<net name="N$5" class="0">
+<pinref part="PAD5" gate="1" pin="P"/>
+<wire x1="139.7" y1="53.34" x2="139.7" y2="63.5" width="0.1524" layer="91"/>
+<label x="114.3" y="63.5" size="1.778" layer="95"/>
+</segment>
+</net>
+<net name="4" class="0">
 <segment>
 <pinref part="ATMEGA328P" gate="G$1" pin="PB3(MOSI/OC2)"/>
 <wire x1="73.66" y1="66.04" x2="144.78" y2="66.04" width="0.1524" layer="91"/>
-<pinref part="15P" gate="G$1" pin="TP"/>
+<pinref part="PAD6" gate="1" pin="P"/>
+<wire x1="144.78" y1="53.34" x2="144.78" y2="66.04" width="0.1524" layer="91"/>
+<label x="114.3" y="66.04" size="1.778" layer="95"/>
 </segment>
 </net>
@@
 <wire x1="129.54" y1="58.42" x2="81.28" y2="58.42" width="0.1524" layer="91"/>
 <label x="81.28" y="58.42" size="1.778" layer="95"/>
-<pinref part="RST" gate="G$1" pin="TP"/>
+<pinref part="PAD8" gate="1" pin="P"/>
+<wire x1="129.54" y1="53.34" x2="129.54" y2="58.42" width="0.1524" layer="91"/>
 </segment>
 </net>
@@
 <wire x1="73.66" y1="96.52" x2="96.52" y2="96.52" width="0.1524" layer="91"/>
 <pinref part="ATMEGA328P" gate="G$1" pin="PD0(RXD)"/>
-<pinref part="RX" gate="G$1" pin="TP"/>
+<pinref part="PAD3" gate="1" pin="P"/>
+<wire x1="96.52" y1="86.36" x2="96.52" y2="96.52" width="0.1524" layer="91"/>
 </segment>
 </net>
@@
 <wire x1="73.66" y1="93.98" x2="91.44" y2="93.98" width="0.1524" layer="91"/>
 <pinref part="ATMEGA328P" gate="G$1" pin="PD1(TXD)"/>
-<pinref part="TX" gate="G$1" pin="TP"/>
-</segment>
-</net>
+<pinref part="PAD2" gate="1" pin="P"/>
+<wire x1="91.44" y1="86.36" x2="91.44" y2="93.98" width="0.1524" layer="91"/>
+</segment>
+</net>
