File: Schematics/baseStation/PCB_baseStation.sch (EAGLE design)
At the start: 42 parts, among them U1 ATMEGA328P, U2 MCP1824ST-3302E/DB, Y2 16MHz

Commit message: Base Station PCB Improvements
Base_SP 1.5
- Fix: connected Regulator for XBee to GND
Connections:
- removed net N$12: U2.GND_(TAB), U2.GND_(TAB)_2
- net GND: now also U2.GND_(TAB), U2.GND_(TAB)_2
Changed lines of the file:
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@@
-</segment>
-</net>
-<net name="N$12" class="0">
-<segment>
-<pinref part="U2" gate="A" pin="GND_(TAB)_2"/>
-<wire x1="104.14" y1="33.02" x2="91.44" y2="33.02" width="0.1524" layer="91"/>
-<wire x1="91.44" y1="33.02" x2="91.44" y2="35.56" width="0.1524" layer="91"/>
-<pinref part="U2" gate="A" pin="GND_(TAB)"/>
-<wire x1="91.44" y1="35.56" x2="91.44" y2="53.34" width="0.1524" layer="91"/>
-<wire x1="104.14" y1="35.56" x2="91.44" y2="35.56" width="0.1524" layer="91"/>
-<junction x="91.44" y="35.56"/>
 </segment>
 </net>
@@
 <wire x1="-91.44" y1="38.1" x2="-91.44" y2="30.48" width="0.1524" layer="91"/>
 </segment>
+<segment>
+<pinref part="U2" gate="A" pin="GND_(TAB)_2"/>
+<wire x1="104.14" y1="33.02" x2="91.44" y2="33.02" width="0.1524" layer="91"/>
+<wire x1="91.44" y1="33.02" x2="91.44" y2="35.56" width="0.1524" layer="91"/>
+<pinref part="U2" gate="A" pin="GND_(TAB)"/>
+<wire x1="91.44" y1="35.56" x2="91.44" y2="53.34" width="0.1524" layer="91"/>
+<wire x1="104.14" y1="35.56" x2="91.44" y2="35.56" width="0.1524" layer="91"/>
+<junction x="91.44" y="35.56"/>
+</segment>
 </net>
